File: KiCAD/TrainTrackr_sh2.kicad_sch (KiCad schematic)
At the start: 0 parts

Commit message: updated sch
Parts:
- added U1, U10, U11, U12, U13, U14, U15, U16, U17, U18, U19, U2, U20, U21, U22, U23, U24, U25, U26, U27, U28, U29, U3, U30, U31, U32, U33, U34, U4, U5, U6, U7, U8, U9: FZ2812-5050, TrainTrackr-footprints:LED_FZ2812-5050, symbol TrainTrackr-lib:FZ2812-5050
Connections:
- new net: U28.2 (DIN), U30.4 (DOUT)
- new net: U26.2 (DIN), U28.4 (DOUT)
- new net: U7.4 (DOUT), U9.2 (DIN)
- new net: U11.2 (DIN), U9.4 (DOUT)
- new net: U14.2 (DIN), U16.4 (DOUT)
- new net: U12.2 (DIN), U14.4 (DOUT)
- new net: U6.2 (DIN), U8.4 (DOUT)
- new net: U4.2 (DIN), U6.4 (DOUT)
- new net: U10.4 (DOUT), U8.2 (DIN)
- new net: U5.4 (DOUT), U7.2 (DIN)
- new net: U11.4 (DOUT), U13.2 (DIN)
- new net: U13.4 (DOUT), U15.2 (DIN)
- new net: U30.2 (DIN), U32.4 (DOUT)
- new net: U22.2 (DIN), U24.4 (DOUT)
- new net: U20.2 (DIN), U22.4 (DOUT)
- new net: U24.2 (DIN), U26.4 (DOUT)
- new net: U17.4 (DOUT), U19.2 (DIN)
- new net: U31.4 (DOUT), U33.2 (DIN)
- new net: U25.4 (DOUT), U27.2 (DIN)
- new net: U27.4 (DOUT), U29.2 (DIN)
- new net: U23.4 (DOUT), U25.2 (DIN)
- new net: U10.2 (DIN), U12.4 (DOUT)
- new net: U32.2 (DIN), U34.4 (DOUT)
- new net: U3.4 (DOUT), U5.2 (DIN)
- new net: U2.2 (DIN), U4.4 (DOUT)
- new net: U29.4 (DOUT), U31.2 (DIN)
- new net: U19.4 (DOUT), U21.2 (DIN)
- new net: U18.2 (DIN), U20.4 (DOUT)
- new net: U21.4 (DOUT), U23.2 (DIN)
- new net: U1.4 (DOUT), U3.2 (DIN)
- new net +5V: U1.3 (VDD), U10.3 (VDD), U11.3 (VDD), U12.3 (VDD), U13.3 (VDD), U14.3 (VDD), U15.3 (VDD), U16.3 (VDD), U17.3 (VDD), U18.3 (VDD), U19.3 (VDD), U2.3 (VDD), U20.3 (VDD), U21.3 (VDD), U22.3 (VDD), U23.3 (VDD), U24.3 (VDD), U25.3 (VDD), U26.3 (VDD), U27.3 (VDD), U28.3 (VDD), U29.3 (VDD), U3.3 (VDD), U30.3 (VDD), U31.3 (VDD), U32.3 (VDD), U33.3 (VDD), U34.3 (VDD), U4.3 (VDD), U5.3 (VDD), U6.3 (VDD), U7.3 (VDD), U8.3 (VDD), U9.3 (VDD)
- new net GND: U1.1 (VSS), U10.1 (VSS), U11.1 (VSS), U12.1 (VSS), U13.1 (VSS), U14.1 (VSS), U15.1 (VSS), U16.1 (VSS), U17.1 (VSS), U19.1 (VSS), U2.1 (VSS), U20.1 (VSS), U21.1 (VSS), U22.1 (VSS), U23.1 (VSS), U24.1 (VSS), U25.1 (VSS), U26.1 (VSS), U27.1 (VSS), U28.1 (VSS), U29.1 (VSS), U3.1 (VSS), U30.1 (VSS), U31.1 (VSS), U32.1 (VSS), U33.1 (VSS), U34.1 (VSS), U4.1 (VSS), U5.1 (VSS), U6.1 (VSS), U7.1 (VSS), U8.1 (VSS), U9.1 (VSS)
- new net Jenk_inbound: U15.4 (DOUT), U17.2 (DIN)
- new net Jenk_outbound: U16.2 (DIN), U18.4 (DOUT)
- new net Pennbrook_INBOUND: U33.4 (DOUT)
- new net Pennbrook_OUTBOUND: U34.2 (DIN)
Other:
- note added: "30th Street Station"
- note added: "Ambler"
- note added: "FRTC"
- note added: "Fort Washington"
- note added: "Glenside"
- note added: "Gwynedd Valley"
- note added: "Jefferson Station"
- note added: "Jenkintown-Wyncote"
- note added: "North Broad"
- note added: "North Hills"
- note added: "North Wales"
- note added: "Oreland"
- note added: "Penllyn"
- note added: "Pennbrook"
- note added: "Suburban Station"
- note added: "Temple University Station"
- note added: "Wayne Junction"
- title: (none) -> Lansdale Doylestown Line LED Array

Commit message: updated layout and sch
Parts:
- removed U1, U10, U11, U12, U13, U14, U15, U16, U17, U18, U19, U2, U20, U21, U22, U23, U24, U25, U26, U27, U28, U29, U3, U30, U31, U32, U33, U34, U4, U5, U6, U7, U8, U9: FZ2812-5050, TrainTrackr-footprints:LED_FZ2812-5050, symbol TrainTrackr-lib:FZ2812-5050
- added D1, D10, D11, D12, D13, D14, D15, D16, D17, D18, D19, D2, D20, D21, D22, D23, D24, D25, D26, D27, D28, D29, D3, D30, D31, D32, D33, D34, D4, D5, D6, D7, D8, D9: IN-PI33TBTPRPGPB, TrainTrackr-footprints:LED_IN-PI33TBTPRPGPB, symbol TrainTrackr-lib:IN-PI33TBTPRPGPB
- added R1, R2: R_US, Resistor_SMD:R_0603_1608Metric_Pad0.98x0.95mm_HandSolder, symbol Device:R_US
Connections:
- net +5V: now also D1.3 (VDD), D10.3 (VDD), D11.3 (VDD), D12.3 (VDD), D13.3 (VDD), D14.3 (VDD), D15.3 (VDD), D16.3 (VDD), D17.3 (VDD), D18.3 (VDD), D19.3 (VDD), D2.3 (VDD), D20.3 (VDD), D21.3 (VDD), D22.3 (VDD), D23.3 (VDD), D24.3 (VDD), D25.3 (VDD), D26.3 (VDD), D27.3 (VDD), D28.3 (VDD), D29.3 (VDD), D3.3 (VDD), D30.3 (VDD), D31.3 (VDD), D32.3 (VDD), D33.3 (VDD), D34.3 (VDD), D4.3 (VDD), D5.3 (VDD), D6.3 (VDD), D7.3 (VDD), D8.3 (VDD), D9.3 (VDD)
- net GND: now also D1.1 (GND), D10.1 (GND), D11.1 (GND), D12.1 (GND), D13.1 (GND), D14.1 (GND), D15.1 (GND), D16.1 (GND), D17.1 (GND), D18.1 (GND), D19.1 (GND), D2.1 (GND), D20.1 (GND), D21.1 (GND), D22.1 (GND), D23.1 (GND), D24.1 (GND), D25.1 (GND), D26.1 (GND), D27.1 (GND), D28.1 (GND), D29.1 (GND), D3.1 (GND), D30.1 (GND), D31.1 (GND), D32.1 (GND), D33.1 (GND), D34.1 (GND), D4.1 (GND), D5.1 (GND), D6.1 (GND), D7.1 (GND), D8.1 (GND), D9.1 (GND), R2.1
- net Pennbrook_INBOUND: now also D33.4 (DOUT)
- net Pennbrook_OUTBOUND: now also D34.2 (DIN)
- new net: D10.2 (DIN), D12.4 (DOUT)
- new net: D10.4 (DOUT), D8.2 (DIN)
- new net: D29.4 (DOUT), D31.2 (DIN)
- new net: D31.4 (DOUT), D33.2 (DIN)
- new net: D23.4 (DOUT), D25.2 (DIN)
- new net: D25.4 (DOUT), D27.2 (DIN)
- new net: D18.2 (DIN), D20.4 (DOUT)
- new net: D16.2 (DIN), D18.4 (DOUT)
- new net: D22.2 (DIN), D24.4 (DOUT)
- new net: D20.2 (DIN), D22.4 (DOUT)
- new net: D17.4 (DOUT), D19.2 (DIN)
- new net: D19.4 (DOUT), D21.2 (DIN)
- new net: D1.2 (DIN), R1.2
- new net: D1.4 (DOUT), D3.2 (DIN)
- new net: D12.2 (DIN), D14.4 (DOUT)
- new net: D11.2 (DIN), D9.4 (DOUT)
- new net: D11.4 (DOUT), D13.2 (DIN)
- new net: D4.2 (DIN), D6.4 (DOUT)
- new net: D2.2 (DIN), D4.4 (DOUT)
- new net: D3.4 (DOUT), D5.2 (DIN)
- new net: D24.2 (DIN), D26.4 (DOUT)
- new net: D30.2 (DIN), D32.4 (DOUT)
- new net: D28.2 (DIN), D30.4 (DOUT)
- new net: D14.2 (DIN), D16.4 (DOUT)
- new net: D13.4 (DOUT), D15.2 (DIN)
- new net: D15.4 (DOUT), D17.2 (DIN)
- new net: D26.2 (DIN), D28.4 (DOUT)
- new net: D21.4 (DOUT), D23.2 (DIN)
- new net: D27.4 (DOUT), D29.2 (DIN)
- new net: D32.2 (DIN), D34.4 (DOUT)
- new net: D2.4 (DOUT), R2.2
- new net: D7.4 (DOUT), D9.2 (DIN)
- new net: D6.2 (DIN), D8.4 (DOUT)
- new net: D5.4 (DOUT), D7.2 (DIN)
- new net DATA_IN: R1.1
