File: KiCAD/TrainTrackr_sh3.kicad_sch (KiCad schematic)
At the start: 18 parts, among them U35 FZ2812-5050, U36 FZ2812-5050, U37 FZ2812-5050, U38 FZ2812-5050, U39 FZ2812-5050, U40 FZ2812-5050, U41 FZ2812-5050, U42 FZ2812-5050, U43 FZ2812-5050, U44 FZ2812-5050, U45 FZ2812-5050, U46 FZ2812-5050, U47 FZ2812-5050, U48 FZ2812-5050, U49 FZ2812-5050, U50 FZ2812-5050, U51 FZ2812-5050, U52 FZ2812-5050

Commit message: updated layout and sch
Parts:
- removed U35, U36, U37, U38, U39, U40, U41, U42, U43, U44, U45, U46, U47, U48, U49, U50, U51, U52: FZ2812-5050, TrainTrackr-footprints:LED_FZ2812-5050, symbol TrainTrackr-lib:FZ2812-5050
- added D35, D36, D37, D38, D39, D40, D41, D42, D43, D44, D45, D46, D47, D48, D49, D50, D51, D52: IN-PI33TBTPRPGPB, TrainTrackr-footprints:LED_IN-PI33TBTPRPGPB, symbol TrainTrackr-lib:IN-PI33TBTPRPGPB
Connections:
- net +5V: now also D35.3 (VDD), D36.3 (VDD), D37.3 (VDD), D38.3 (VDD), D39.3 (VDD), D40.3 (VDD), D41.3 (VDD), D42.3 (VDD), D43.3 (VDD), D44.3 (VDD), D45.3 (VDD), D46.3 (VDD), D47.3 (VDD), D48.3 (VDD), D49.3 (VDD), D50.3 (VDD), D51.3 (VDD), D52.3 (VDD)
- net GND: now also D35.1 (GND), D36.1 (GND), D37.1 (GND), D38.1 (GND), D39.1 (GND), D40.1 (GND), D41.1 (GND), D42.1 (GND), D43.1 (GND), D44.1 (GND), D45.1 (GND), D46.1 (GND), D47.1 (GND), D48.1 (GND), D49.1 (GND), D50.1 (GND), D51.1 (GND), D52.1 (GND)
- net Pennbrook_INBOUND: now also D35.2 (DIN)
- net Pennbrook_OUTBOUND: now also D36.4 (DOUT)
- new net: D44.2 (DIN), D46.4 (DOUT)
- new net: D42.2 (DIN), D44.4 (DOUT)
- new net: D38.2 (DIN), D40.4 (DOUT)
- new net: D36.2 (DIN), D38.4 (DOUT)
- new net: D51.4 (DOUT), D52.2 (DIN)
- new net: D50.2 (DIN), D52.4 (DOUT)
- new net: D45.4 (DOUT), D47.2 (DIN)
- new net: D47.4 (DOUT), D49.2 (DIN)
- new net: D39.4 (DOUT), D41.2 (DIN)
- new net: D41.4 (DOUT), D43.2 (DIN)
- new net: D48.2 (DIN), D50.4 (DOUT)
- new net: D35.4 (DOUT), D37.2 (DIN)
- new net: D49.4 (DOUT), D51.2 (DIN)
- new net: D46.2 (DIN), D48.4 (DOUT)
- new net: D37.4 (DOUT), D39.2 (DIN)
- new net: D40.2 (DIN), D42.4 (DOUT)
- new net: D43.4 (DOUT), D45.2 (DIN)
