File: KiCAD/TrainTrackr_sh4.kicad_sch (KiCad schematic)
At the start: 1 part

Commit message: silk screen png and sch updates
Parts:
- added J1: 54-00165, 54-00165:TENSILITY_54-00165, symbol TrainTrackr-lib:54-00165
Changed lines of the file:
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@@
+		)
+	)
+	(symbol
+		(lib_id "TrainTrackr-lib:54-00165")
+		(at 323.85 73.66 0)
+		(unit 1)
+		(exclude_from_sim no)
+		(in_bom yes)
+		(on_board yes)
+		(dnp no)
+		(fields_autoplaced yes)
+		(property "Reference" "J1"
+			(at 319.0903 64.77 0)
+			(effects
+				(font
+					(size 1.27 1.27)
+				)
+			)
+		)
+		(property "Value" "54-00165"
+			(at 319.0903 67.31 0)
+			(effects
+				(font
+					(size 1.27 1.27)
+				)
+			)
+		)
+		(property "Footprint" "54-00165:TENSILITY_54-00165"
+			(at 325.374 65.278 0)
+			(effects
+				(font
+					(size 1.27 1.27)
+				)
+				(justify bottom)
+				(hide yes)
+			)
+		)
+		(property "Datasheet" "https://tensility.s3.us-west-2.amazonaws.com/uploads/pdffiles/54-00165.pdf"
+			(at 323.85 73.66 0)
+			(effects
+				(font
+					(size 1.27 1.27)
+				)
+				(hide yes)
+			)
+		)
+		(property "Description" ""
+			(at 323.85 73.66 0)
+			(effects
+				(font
+					(size 1.27 1.27)
+				)
+				(hide yes)
+			)
+		)
+		(property "PARTREV" "A"
+			(at 323.85 73.66 0)
+			(effects
+				(font
+					(size 1.27 1.27)
+				)
+				(justify bottom)
+				(hide yes)
+			)
+		)
+		(property "MANUFACTURER" "TENSILITY"
+			(at 314.452 61.468 0)
+			(effects
+				(font
+					(size 1.27 1.27)
+				)
+				(justify bottom)
+				(hide yes)
+			)
+		)
+		(property "SNAPEDA_PN" "54-00164"
+			(at 314.198 59.436 0)
+			(effects
+				(font
+					(size 1.27 1.27)
+				)
+				(justify bottom)
+				(hide yes)
+			)
+		)
+		(property "MAXIMUM_PACKAGE_HEIGHT" "11.3mm"
+			(at 314.198 63.246 0)
+			(effects
+				(font
+					(size 1.27 1.27)
+				)
+				(justify bottom)
+				(hide yes)
+			)
+		)
+		(property "STANDARD" "Manufacturer Recommendations"
+			(at 325.374 65.278 0)
+			(effects
+				(font
+					(size 1.27 1.27)
+				)
+				(justify bottom)
+				(hide yes)
+			)
+		)
+		(pin "A1"
+		)
+		(pin "C"
+		)
+		(pin "B"
+		)
+		(pin "A2"
+		)
+		(instances
+			(project ""
+				(path "/779c311e-6596-48d7-a471-956474340a54/849774d0-25f0-4453-9479-ecac56d96414"
+					(reference "J1")
+					(unit 1)
+				)
+			)
 		)
 	)

Commit message: updated layout and sch
Parts:
- added Q1: DMG2305UX-13, TrainTrackr-footprints:train, symbol TrainTrackr-lib:DMG2305UX-13
- added U1: SN74LV1T34DCKR, TrainTrackr-footprints:DCK0005A_L, symbol TrainTrackr-lib:SN74LV1T34DCKR
- J1: footprint 54-00165:TENSILITY_54-00165 -> TrainTrackr-footprints:TENSILITY_54-00165
Connections:
- net GND: now reaches A1.13 (GND), A1.18 (GND), A1.23 (GND), A1.28 (GND), A1.3 (GND), A1.38 (GND), A1.8 (GND)
- net GND: now also A1.33 (AGND), J1.B, J1.C, U1.3 (GND)
- net at A1.24 (GPIO18): now also U1.2 (A)
- net at A1.39 (VSYS): now also Q1.2
- net at A1.40 (VBUS): now also Q1.1
- net +5V: now reaches J1.A1
- net +5V: now also J1.A2, Q1.3, U1.5 (VCC)
- new net DATA_IN: U1.4 (Y)
Other:
- moved on the sheet: J1
