File: KiCAD/TrainTrackr.kicad_pcb (KiCad board)
At the start: 2 copper layers, 203.2 x 254 mm, 59 parts, among them J1 54-00165, Q1 DMG2305UX-13, U1 SN74LV1T34DCKR

Commit message: sch layout update
Parts:
- moved J1 76.2 mm to (319.7, 221.4)
- moved U1 65.8 mm to (375.3, 353.9)
Routing:
- net +5V: track 679.7 -> 975.8 mm
- net Net-(A1-GPIO18): track 0.00 -> 108.8 mm
- net DATA_IN: track 0.00 -> 2.69 mm
- net GND: vias 21 -> 59
- added copper zone on B.Cu, net GND
- added copper zone on F.Cu, net GND
